File: canbus_pic18_adapter.kicad_pcb (KiCad board)
At the start: 2 copper layers, 58.8 x 32 mm, 15 parts, among them J1 Conn_01x06_Socket, J2 Conn_01x14_Pin, J3 Conn_01x14_Pin, J4 Conn_01x05_Pin, U1 PIC18F2XK80, Y1 10Mhz

Commit message: pass DRC
Routing:
- net GND: vias 1 -> 3
Changed lines of the file:
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@@
 		(tags "Through hole pin header THT 1x14 2.54mm single row")
 		(property "Reference" "J2"
-			(at 0 -2.33 270)
+			(at 0 -2.33 -90)
 			(layer "F.SilkS")
 			(effects
@@
 		)
 		(property "Value" "Conn_01x14_Pin"
-			(at 0 35.35 270)
+			(at 0 35.35 -90)
 			(layer "F.Fab")
 			(effects
@@
 		)
 		(fp_text user "${REFERENCE}"
-			(at 0 16.51 360)
+			(at 0 16.51 0)
 			(layer "F.Fab")
 			(effects
@@
 		)
 		(fp_text user "${REFERENCE}"
-			(at -5.775 6.35 270)
+			(at -5.775 6.35 -90)
 			(layer "F.Fab")
 			(effects
@@
 		(tags "C Disc series Radial pin pitch 2.50mm  diameter 3.4mm width 2.1mm Capacitor")
 		(property "Reference" "C4"
-			(at 1.25 -2.3 360)
+			(at 1.25 -2.3 0)
 			(layer "F.SilkS")
 			(effects
@@
 		)
 		(property "Value" "22pF"
-			(at 1.25 2.3 360)
+			(at 1.25 2.3 0)
 			(layer "F.Fab")
 			(effects
@@
 		)
 		(fp_text user "${REFERENCE}"
-			(at 1.25 0 360)
+			(at 1.25 0 0)
 			(layer "F.Fab")
 			(effects
@@
 		(tags "LED diameter 3.0mm 2 pins")
 		(property "Reference" "D1"
-			(at 1.27 -2.96 270)
+			(at 1.27 -2.96 -90)
 			(layer "F.SilkS")
 			(effects
@@
 		)
 		(property "Value" "LED"
-			(at 1.27 2.96 270)
+			(at 1.27 2.96 -90)
 			(layer "F.Fab")
 			(effects
@@
 		(tags "Through hole pin header THT 1x14 2.54mm single row")
 		(property "Reference" "J3"
-			(at 0 -2.33 270)
+			(at 0 -2.33 -90)
 			(layer "F.SilkS")
 			(effects
@@
 		)
 		(property "Value" "Conn_01x14_Pin"
-			(at 0 35.35 270)
+			(at 0 35.35 -90)
 			(layer "F.Fab")
 			(effects
@@
 		)
 		(fp_text user "${REFERENCE}"
-			(at 0 16.51 360)
+			(at 0 16.51 0)
 			(layer "F.Fab")
 			(effects
@@
 		(tags "THT DIP DIL PDIP 2.54mm 7.62mm 300mil Socket")
 		(property "Reference" "U1"
-			(at 3.81 -2.33 270)
+			(at 3.81 -2.33 -90)
 			(layer "F.SilkS")
 			(effects
@@
 		)
 		(property "Value" "PIC18F2XK80"
-			(at 3.81 35.35 270)
+			(at 3.81 35.35 -90)
 			(layer "F.Fab")
 			(effects
@@
 		)
 		(fp_text user "${REFERENCE}"
-			(at 3.81 16.51 270)
+			(at 3.81 16.51 -90)
 			(layer "F.Fab")
 			(effects
@@
 		(tags "capacitor handsolder")
 		(property "Reference" "C1"
-			(at 0 1.68 360)
+			(at 0 1.68 0)
 			(layer "B.SilkS")
 			(effects
@@
 		)
 		(property "Value" "10uF"
-			(at 0 -1.68 360)
+			(at 0 -1.68 0)
 			(layer "B.Fab")
 			(effects
@@
 		)
 		(fp_text user "${REFERENCE}"
-			(at 0 0 360)
+			(at 0 0 0)
 			(layer "B.Fab")
 			(effects
@@
 	)
 	(via
+		(at 93.98 114.3)
+		(size 0.8)
+		(drill 0.4)
+		(layers "F.Cu" "B.Cu")
+		(free yes)
+		(net 2)
+	)
+	(via
 		(at 122.809 91.313)
 		(size 0.8)
@@
 		(net 2)
 	)
+	(via
+		(at 92.964 85.979)
+		(size 0.8)
+		(drill 0.4)
+		(layers "F.Cu" "B.Cu")
+		(free yes)
+		(net 2)
+	)
 	(segment
 		(start 124.149 103.067)
@@
 			(clearance 0.2)
 		)
-		(min_thickness 0.2)
+		(min_thickness 0.21)
 		(filled_areas_thickness no)
 		(fill yes
